File: Driver Motor PaP_V2.0/Driver Motor PaP_V2.0.sch (KiCad schematic (older format))
At the start: 15 parts

Commit message: se empezo agregar footprints y continuar
Parts:
- removed J?: Conn_01x02, symbol Connector_Generic:Conn_01x02
- removed U? (x6): LM358, symbol Amplifier_Operational:LM358
- added C1, C2, C3: 100nF, Capacitor_THT:C_Disc_D4.3mm_W1.9mm_P5.00mm, symbol Device:C
- added D1: LED_PWR, LED_THT:LED_D5.0mm, symbol Device:LED_ALT
- added J3, J4: Conn_01x04, symbol Connector_Generic:Conn_01x04
- added J5: Conn_01x01, symbol Connector_Generic:Conn_01x01
- added J6, J7: Conn_01x02, symbol Connector_Generic:Conn_01x02
- added Q1: BC547, Package_TO_SOT_THT:TO-92_Inline, symbol Transistor_BJT:BC547
- added R1: 220, symbol Device:R
- added R2: 33k, symbol Device:R
- added R3: 470, symbol Device:R
- added U1, U2, U3: LM358, symbol Amplifier_Operational:LM358
- C4: renamed from C?; value CP1 -> 100nF; footprint (none) -> Capacitor_THT:C_Disc_D4.3mm_W1.9mm_P5.00mm
- gave numbers to parts that had none: 7
Connections:
- net GND: now also A1.1 (GND), C1.2, C2.2, C3.2, J3.1 (Pin_1), Q1.3 (E), R1.2, U1.4 (V-), U2.4 (V-), U3.4 (V-)
- net GNDPWR: now also A1.7 (GND), C4.2
- net VCC: now also A1.13 (~RST), A1.14 (~SLP), C1.1, C2.1, C3.1, D1.2 (A), R3.1, U1.8 (V+), U2.8 (V+), U3.8 (V+)
- net VDD: now also A1.8 (VMOT), C4.1
- net at A1.10 (M0): now also U2.1, U2.2 (-)
- net at A1.11 (M1): now also U2.6 (-), U2.7
- net at A1.12 (M2): now also U3.1, U3.2 (-)
- net at A1.15 (STEP): now also U1.1, U1.2 (-)
- net at A1.16 (DIR): now also U1.6 (-), U1.7
- net at A1.3 (A2): now also J6.2 (Pin_2)
- net at A1.4 (A1): now also J6.1 (Pin_1)
- net at A1.5 (B1): now also J7.1 (Pin_1)
- net at A1.6 (B2): now also J7.2 (Pin_2)
- net at A1.9 (~EN): now also Q1.1 (C), R3.2
- new net: Q1.2 (B), R2.1
- new net: J3.4 (Pin_4), R2.2
- new net: J3.3 (Pin_3), U1.3 (+)
- new net: J3.2 (Pin_2), U1.5 (+)
- new net: J4.4 (Pin_4), U2.3 (+)
- new net: J4.3 (Pin_3), U2.5 (+)
- new net: J4.2 (Pin_2), U3.3 (+)
- new net: J4.1 (Pin_1), U3.5 (+)
- new net: J5.1 (Pin_1), U3.6 (-), U3.7
- new net: D1.1 (K), R1.1
- no-connect marks 0 -> 1
Other:
- note added: "4 - Enable\n3 - Step\n2 - Dir \n1 - GND (de la CIAA)"
- note added: "4 - M0\n3 - M1\n2 - M2\n1 - Seguidor de \n tensión libre"
- note added: "Compuerta NOT para habilitar \nMotor PaP"
- note added: "Conexión al motor bipolar de 4 hilos\n"
- moved on the sheet: A1, C4

Commit message: esquematico Finalizado e iniciando el ruteo en el PCB
Parts:
- added J8: Conn_01x01, Connector_PinHeader_2.54mm:PinHeader_1x01_P2.54mm_Vertical, symbol Connector_Generic:Conn_01x01
- added JP1, JP2, JP3, JP4, JP5, JP6: Jumper_2_Open, Connector_PinHeader_2.54mm:PinHeader_1x02_P2.54mm_Vertical, symbol Jumper:Jumper_2_Open
- C4: footprint Capacitor_THT:C_Disc_D4.3mm_W1.9mm_P5.00mm -> Capacitor_THT:CP_Radial_D10.0mm_P2.50mm
- H1, H2, H3, H4: footprint (none) -> MountingHole:MountingHole_4mm_Pad_Via
- J1, J2: footprint (none) -> TerminalBlock_Phoenix:TerminalBlock_Phoenix_MKDS-1,5-2-5.08_1x02_P5.08mm_Horizontal
- J3, J4: footprint (none) -> Connector_Molex:Molex_KK-254_AE-6410-04A_1x04_P2.54mm_Vertical
- J5: footprint (none) -> Connector_PinHeader_2.54mm:PinHeader_1x01_P2.54mm_Vertical
- J6, J7: footprint (none) -> Connector_Molex:Molex_KK-254_AE-6410-02A_1x02_P2.54mm_Vertical
- R1, R2, R3: footprint (none) -> Resistor_THT:R_Axial_DIN0207_L6.3mm_D2.5mm_P10.16mm_Horizontal
- U1, U2, U3: footprint (none) -> Package_DIP:DIP-8_W7.62mm_Socket
Connections:
- net GND: now also JP3.1 (A), JP5.2 (B)
- net VCC: now also JP1.1 (A), JP4.2 (B)
- net at U2.6 (-), U2.7: now also JP2.1 (A); no longer A1.11 (M1)
- net at U3.1, U3.2 (-): now also JP6.2 (B); no longer A1.12 (M2)
- net at A1.2 (~FLT): now also J8.1 (Pin_1)
- net at A1.5 (B1): now also J7.2 (Pin_2); no longer J7.1 (Pin_1)
- net at A1.6 (B2): now also J7.1 (Pin_1); no longer J7.2 (Pin_2)
- new net: A1.11 (M1), JP1.2 (B), JP2.2 (B), JP3.2 (B)
- new net: A1.12 (M2), JP4.1 (A), JP5.1 (A), JP6.1 (A)
- no-connect marks 1 -> 0

Commit message: Finalizado el ruteo. Revisar nuevamente
Parts:
- C4: footprint Capacitor_THT:CP_Radial_D10.0mm_P2.50mm -> Capacitor_THT:CP_Radial_D6.3mm_P2.50mm
Changed lines of the file:
@@
 encoding utf-8
 Sheet 1 1
-Title "Driver Motor Paso a Paso - Simple Faz"
+Title "Driver Motor Paso a Paso - Doble Faz"
 Date "2020-05-17"
 Rev "2.0"
@@
 F 0 "C4" H 8065 2496 50  0000 L CNN
 F 1 "100nF" H 8065 2405 50  0000 L CNN
-F 2 "Capacitor_THT:CP_Radial_D10.0mm_P2.50mm" H 7950 2450 50  0001 C CNN
+F 2 "Capacitor_THT:CP_Radial_D6.3mm_P2.50mm" H 7950 2450 50  0001 C CNN
 F 3 "~" H 7950 2450 50  0001 C CNN
 	1    7950 2450
@@
 Alimentación Motor\n(8,2 v - 45 v)
 $Comp
-L Transistor_BJT:BC547 Q1
-U 1 1 5EC2EF50
-P 5750 1650
-F 0 "Q1" H 5941 1696 50  0000 L CNN
-F 1 "BC547" H 5941 1605 50  0000 L CNN
-F 2 "Package_TO_SOT_THT:TO-92_Inline" H 5950 1575 50  0001 L CIN
-F 3 "http://www.fairchildsemi.com/ds/BC/BC547.pdf" H 5750 1650 50  0001 L CNN
-	1    5750 1650
-	1    0    0    -1
-$EndComp
-$Comp
 L Device:R R3
 U 1 1 5EC341B0
@@
 Wire Wire Line
 	7550 3400 8200 3400
+$Comp
+L Transistor_BJT:BC547 Q1
+U 1 1 5ED0DF68
+P 5750 1650
+F 0 "Q1" H 5941 1696 50  0000 L CNN
+F 1 "BC547" H 5941 1605 50  0000 L CNN
+F 2 "Package_TO_SOT_THT:TO-92_Inline" H 5950 1575 50  0001 L CIN
+F 3 "http://www.fairchildsemi.com/ds/BC/BC547.pdf" H 5750 1650 50  0001 L CNN
+	1    5750 1650
+	1    0    0    -1
+$EndComp
 $EndSCHEMATC

Commit message: Cambiando y creando nuevo Footprints y modelos 3D
Parts:
- C1, C2, C3: footprint Capacitor_THT:C_Disc_D4.3mm_W1.9mm_P5.00mm -> Capacitor_THT:C_Disc_D5.0mm_W2.5mm_P2.50mm
- C4: footprint Capacitor_THT:CP_Radial_D6.3mm_P2.50mm -> Capacitor_THT:C_Radial_D6.3mm_H11.0mm_P2.50mm
- J1, J2: footprint TerminalBlock_Phoenix:TerminalBlock_Phoenix_MKDS-1,5-2-5.08_1x02_P5.08mm_Horizontal -> Terminal Degson:dg126
Changed lines of the file:
@@
 F 0 "J1" H 1300 1050 50  0000 C CNN
 F 1 "Conn_01x02" H 1318 1116 50  0000 C CNN
-F 2 "TerminalBlock_Phoenix:TerminalBlock_Phoenix_MKDS-1,5-2-5.08_1x02_P5.08mm_Horizontal" H 1400 1350 50  0001 C CNN
+F 2 "Terminal Degson:dg126" H 1400 1350 50  0001 C CNN
 F 3 "~" H 1400 1350 50  0001 C CNN
 	1    1400 1350
@@
 F 0 "C4" H 8065 2496 50  0000 L CNN
 F 1 "100nF" H 8065 2405 50  0000 L CNN
-F 2 "Capacitor_THT:CP_Radial_D6.3mm_P2.50mm" H 7950 2450 50  0001 C CNN
+F 2 "Capacitor_THT:C_Radial_D6.3mm_H11.0mm_P2.50mm" H 7950 2450 50  0001 C CNN
 F 3 "~" H 7950 2450 50  0001 C CNN
 	1    7950 2450
@@
 F 0 "J2" H 1318 2475 50  0000 C CNN
 F 1 "Conn_01x02" H 1318 2566 50  0000 C CNN
-F 2 "TerminalBlock_Phoenix:TerminalBlock_Phoenix_MKDS-1,5-2-5.08_1x02_P5.08mm_Horizontal" H 1400 2800 50  0001 C CNN
+F 2 "Terminal Degson:dg126" H 1400 2800 50  0001 C CNN
 F 3 "~" H 1400 2800 50  0001 C CNN
 	1    1400 2800
@@
 F 0 "C2" H 1665 5296 50  0000 L CNN
 F 1 "100nF" H 1665 5205 50  0000 L CNN
-F 2 "Capacitor_THT:C_Disc_D4.3mm_W1.9mm_P5.00mm" H 1588 5100 50  0001 C CNN
+F 2 "Capacitor_THT:C_Disc_D5.0mm_W2.5mm_P2.50mm" H 1588 5100 50  0001 C CNN
 F 3 "~" H 1550 5250 50  0001 C CNN
 	1    1550 5250
@@
 F 0 "C3" H 2565 5296 50  0000 L CNN
 F 1 "100nF" H 2565 5205 50  0000 L CNN
-F 2 "Capacitor_THT:C_Disc_D4.3mm_W1.9mm_P5.00mm" H 2488 5100 50  0001 C CNN
+F 2 "Capacitor_THT:C_Disc_D5.0mm_W2.5mm_P2.50mm" H 2488 5100 50  0001 C CNN
 F 3 "~" H 2450 5250 50  0001 C CNN
 	1    2450 5250
@@
 F 0 "C1" H 765 5246 50  0000 L CNN
 F 1 "100nF" H 765 5155 50  0000 L CNN
-F 2 "Capacitor_THT:C_Disc_D4.3mm_W1.9mm_P5.00mm" H 688 5050 50  0001 C CNN
+F 2 "Capacitor_THT:C_Disc_D5.0mm_W2.5mm_P2.50mm" H 688 5050 50  0001 C CNN
 F 3 "~" H 650 5200 50  0001 C CNN
 	1    650  5200
